File: ATMEGA328P_AU_BootloaderBurner/Schematic/Schematic.kicad_pcb (KiCad board)
At the start: 2 copper layers, 36 x 53 mm, 10 parts, among them J1 Conn_01x16, J2 Conn_01x16, Y1 16MHz

Commit message: Updated component values. Minor silkscreen changes.
Other:
- net class Default removed
- board text added: "ATMEGA328P-AU Bootloader Burner 21_13_0061 retronics.no"
- board text removed: "ATMEGA328P-AU Bootloader Burner 21_13_0061 Bjørner Sandom"
