File: ATMEGA328P_AU_BreadboardAdapter/Schematic/ATMEGA328P_5V_16MHz/ATMEGA328P_5V_16MHz.kicad_sch (KiCad schematic)
At the start: 37 parts, among them J1 Pin header 1, J2 Pin header 2, J3 FTDI, Q1 Si3493DDV, Q2 BC857BS, SW1 RESET, U1 TPS54302, U2 ATMEGA328P-AU, Y1 16MHz 16pF

Commit message: Organized schematic
Parts:
- D1: value "Vcc" -> "5V"
- L1: Comments (none) -> TDK VLS252012HBX-100M-1
Connections:
- net VCC: no longer D1.2 (A), J2.2 (Pin_2), J3.3 (Pin_3), Q1.4 (S), Q2.4 (E2)
- net VDC renamed Vin
- new net +5V: D1.2 (A), J2.2 (Pin_2), J3.3 (Pin_3), Q1.4 (S), Q2.4 (E2)
Other:
- note added: "Interface"
- note added: "MCU"
- note added: "Reverse current protection"
- note added: "Switched voltage regulator"
- moved on the sheet: C10, C11, C12, C7, C8, C9, D3, J1, J2, J3, R10, R11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
